File: pcb/GateLinkMaster.kicad_pcb (KiCad board)
At the start: 2 copper layers, 39 parts, among them J1 Input, J2 Screw_Terminal_01x03, J3 Screw_Terminal_01x03, J4 Screw_Terminal_01x03, J5 Screw_Terminal_01x03, J6 Screw_Terminal_01x02, K2 SANYOU_SRD_Form_C, K3 SANYOU_SRD_Form_C, K4 SANYOU_SRD_Form_C, K5 SANYOU_SRD_Form_C, Q2 MMBT2222A, Q3 MMBT2222A, Q4 MMBT2222A, Q5 MMBT2222A, U3 ESP32-DevKitC

Commit message: Update PCB Layout
Parts:
- added J7: Screw_Terminal_01x08, TerminalBlock_WAGO:TerminalBlock_WAGO_236-108_1x08_P5.00mm_45Degree, F.Cu at (42.5, 91.5)
- added R17: 910, Resistor_SMD:R_0805_2012Metric, F.Cu at (59.1, 66.3)
- added R18: 10k, Resistor_SMD:R_0805_2012Metric, F.Cu at (77.5, 61.5)
- added R19: 910, Resistor_SMD:R_0805_2012Metric, F.Cu at (54.6, 71.3)
- added R20: 910, Resistor_SMD:R_0805_2012Metric, F.Cu at (59.1, 71.3)
- added R21: 10k, Resistor_SMD:R_0805_2012Metric, F.Cu at (77.5, 68.5)
- added R22: 910, Resistor_SMD:R_0805_2012Metric, F.Cu at (54.6, 76.3)
- added R23: 910, Resistor_SMD:R_0805_2012Metric, F.Cu at (59.1, 76.3)
- added R24: 10k, Resistor_SMD:R_0805_2012Metric, F.Cu at (77.5, 75.5)
- added R25: 910, Resistor_SMD:R_0805_2012Metric, F.Cu at (54.6, 81.3)
- added R26: 910, Resistor_SMD:R_0805_2012Metric, F.Cu at (59.1, 81.3)
- added R27: 10k, Resistor_SMD:R_0805_2012Metric, F.Cu at (77.5, 82.5)
- added R28: 910, Resistor_SMD:R_0805_2012Metric, F.Cu at (54.6, 86.3)
- added R29: 910, Resistor_SMD:R_0805_2012Metric, F.Cu at (59.1, 86.3)
- added R30: 10k, Resistor_SMD:R_0805_2012Metric, F.Cu at (77.5, 89.5)
- added R31: 910, Resistor_SMD:R_0805_2012Metric, F.Cu at (54.6, 56.4)
- added R32: 910, Resistor_SMD:R_0805_2012Metric, F.Cu at (59.1, 56.4)
- added R33: 10k, Resistor_SMD:R_0805_2012Metric, F.Cu at (77.5, 47.5)
- added U1: LTV-356T, Package_SO:SO-4_4.4x3.6mm_P2.54mm, F.Cu at (69.2, 58.6)
- added U2: LTV-356T, Package_SO:SO-4_4.4x3.6mm_P2.54mm, F.Cu at (69.4, 65.6)
- added U4: LTV-356T, Package_SO:SO-4_4.4x3.6mm_P2.54mm, F.Cu at (69.6, 72.6)
- added U5: LTV-356T, Package_SO:SO-4_4.4x3.6mm_P2.54mm, F.Cu at (69.6, 79.6)
- added U6: LTV-356T, Package_SO:SO-4_4.4x3.6mm_P2.54mm, F.Cu at (69.7, 86.6)
- added U7: LTV-356T, Package_SO:SO-4_4.4x3.6mm_P2.54mm, F.Cu at (69.6, 93.6)
- added U8: LTV-356T, Package_SO:SO-4_4.4x3.6mm_P2.54mm, F.Cu at (69.4, 51.6)
- J1: value Input -> GND_Jumper; footprint TerminalBlock:TerminalBlock_MaiXu_MX126-5.0-05P_1x05_P5.00mm -> Connector_PinHeader_2.54mm:PinHeader_1x02_P2.54mm_Vertical
- R1, R16, R2: value 10k -> 910; footprint Resistor_SMD:R_0603_1608Metric -> Resistor_SMD:R_0805_2012Metric
- R3: footprint Resistor_SMD:R_0603_1608Metric -> Resistor_SMD:R_0805_2012Metric
- moved R12 151.4 mm to (245.5, 84.0)
- moved R10 144.0 mm to (241.5, 89.0)
- moved R11 144.0 mm to (241.5, 91.5)
- moved R8 144.0 mm to (241.5, 84.0)
- moved R9 144.0 mm to (241.5, 86.5)
- moved R13 142.4 mm to (245.5, 86.5)
- moved R14 142.4 mm to (245.5, 89.0)
- moved R15 142.4 mm to (245.5, 91.5)
- moved J2 139.4 mm to (179.4, 41.3), turned to 90 degrees
- moved R7 137.1 mm to (237.4, 91.5)
- moved D6 124.4 mm to (188.8, 132.7)
- moved R6 117.9 mm to (139.9, 30.6), turned to -90 degrees
- moved K2 113.9 mm to (151.0, 36.5), turned to 0 degrees
- moved R3 105.8 mm to (77.5, 54.5), turned to -90 degrees
- moved Q2 103.8 mm to (141.9, 38.0)
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Connections:
- J1 pad 1: /IN4 -> GND1
- J1 pad 2: /IN3 -> GND
- R1 pad 1: +3V3 -> Net-(R1-Pad1)
- R1 pad 2: /IN4 -> Net-(R1-Pad2)
- R16 pad 1: +3V3 -> /IN_T_3
- R16 pad 2: /IN1 -> Net-(R16-Pad2)
- R2 pad 1: +3V3 -> /IN_T_2
- R2 pad 2: /IN3 -> Net-(R1-Pad1)
- R3 pad 1: +3V3 -> +5V
- U3 pad 10: unconnected-(U3-DAC_2/ADC2_CH9/GPIO26-Pad10) -> /IN4
- U3 pad 11: unconnected-(U3-ADC2_CH7/GPIO27-Pad11) -> /IN5
- U3 pad 27: /IN4 -> /IN6
- U3 pad 28: /IN3 -> /IN7
- U3 pad 36: /IN2 -> /IN1
- U3 pad 37: /IN1 -> /IN2
- U3 pad 9: unconnected-(U3-DAC_1/ADC2_CH8/GPIO25-Pad9) -> /IN3
Routing:
- net +3V3: track 111.0 -> 0.00 mm, vias 4 -> 0
- net GND1: track 0.00 -> 86.1 mm, vias 0 -> 7
- net /IN7: track 0.00 -> 71.0 mm
- net /IN6: track 0.00 -> 67.5 mm, vias 0 -> 1
- net /SIG2: track 63.5 -> 0.00 mm
- net Net-(J5-Pin_2): track 0.00 -> 29.3 mm
- net Net-(J4-Pin_2): track 0.00 -> 29.1 mm
- net /IN5: track 0.00 -> 28.7 mm
- net Net-(J3-Pin_2): track 0.00 -> 28.6 mm
- net Net-(J5-Pin_1): track 0.00 -> 15.6 mm
- net Net-(J4-Pin_1): track 0.00 -> 15.4 mm
- net Net-(J3-Pin_1): track 0.00 -> 14.9 mm
- net Net-(J5-Pin_3): track 0.00 -> 14.7 mm
- net Net-(J4-Pin_3): track 0.00 -> 14.5 mm
- net Net-(J3-Pin_3): track 0.00 -> 14.4 mm
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- added copper zone on B.Cu, net GND
- added copper zone on B.Cu, net GND1

Commit message: PCB Design
Parts:
- moved J6 112.4 mm to (87.0, 107.5)
- moved R13 109.7 mm to (138.0, 108.5)
- moved R9 106.2 mm to (141.0, 52.0), turned to -90 degrees
- moved R14 105.3 mm to (142.0, 108.5)
- moved R15 105.1 mm to (140.5, 96.0), turned to -90 degrees
- moved R12 104.9 mm to (141.0, 74.5), turned to -90 degrees
- moved R10 104.0 mm to (137.5, 86.5)
- moved R7 103.5 mm to (137.5, 64.5)
- moved R8 101.3 mm to (142.0, 64.5)
- moved R11 99.6 mm to (142.0, 86.5)
- moved D6 89.4 mm to (146.5, 54.0), turned to -90 degrees
- moved Q3 81.0 mm to (142.0, 60.5), turned to 90 degrees
- moved D8 74.5 mm to (146.5, 76.0), turned to -90 degrees
- moved Q4 69.1 mm to (142.0, 82.5), turned to 90 degrees
- moved D7 64.4 mm to (141.0, 78.5), turned to 90 degrees
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Routing:
- net +5V: track 83.5 -> 290.5 mm, vias 7 -> 11
- net GND: track 18.9 -> 141.8 mm, vias 7 -> 12
- net /SIG4: track 0.00 -> 54.0 mm
- net /SIG2: track 0.00 -> 34.4 mm, vias 0 -> 1
- net /SIG3: track 0.00 -> 34.0 mm, vias 0 -> 1
- net Net-(D10-A): track 0.00 -> 23.1 mm
- net Net-(D5-K): track 0.00 -> 22.6 mm
- net Net-(D7-K): track 0.00 -> 22.3 mm
- net /SIG1: track 0.00 -> 17.7 mm, vias 0 -> 1
- net Net-(Q4-B): track 0.00 -> 5.96 mm
- net Net-(Q3-B): track 0.00 -> 5.96 mm
- net Net-(Q5-B): track 0.00 -> 5.53 mm
- net Net-(D7-A): track 0.00 -> 2.39 mm
- net Net-(D5-A): track 0.00 -> 2.39 mm
- net Net-(D9-A): track 0.00 -> 2.17 mm
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Other:
- board outline added: 150.8 x 87.5 mm
