File: pcb/GateLinkMaster.kicad_sch (KiCad schematic)
At the start: 39 parts, among them J1 Input, J2 Screw_Terminal_01x03, J3 Screw_Terminal_01x03, J4 Screw_Terminal_01x03, J5 Screw_Terminal_01x03, J6 Screw_Terminal_01x02, K2 SANYOU_SRD_Form_C, K3 SANYOU_SRD_Form_C, K4 SANYOU_SRD_Form_C, K5 SANYOU_SRD_Form_C, Q2 MMBT2222A, Q3 MMBT2222A, Q4 MMBT2222A, Q5 MMBT2222A, U3 ESP32-DevKitC

Commit message: Update PCB Layout
Parts:
- removed J1: Input, TerminalBlock:TerminalBlock_MaiXu_MX126-5.0-05P_1x05_P5.00mm, symbol Connector:Screw_Terminal_01x05
- added J1: GND_Jumper, Connector_PinHeader_2.54mm:PinHeader_1x02_P2.54mm_Vertical, symbol Connector:Conn_01x02_Pin
- added J7: Screw_Terminal_01x08, TerminalBlock_WAGO:TerminalBlock_WAGO_236-108_1x08_P5.00mm_45Degree, symbol Connector:Screw_Terminal_01x08
- added R17, R19, R20, R22, R23, R25, R26, R28, R29, R31, R32: 910, Resistor_SMD:R_0805_2012Metric, symbol Device:R
- added R18, R21, R24, R27, R30, R33: 10k, Resistor_SMD:R_0805_2012Metric, symbol Device:R
- added U1, U2, U4, U5, U6, U7, U8: LTV-356T, Package_SO:SO-4_4.4x3.6mm_P2.54mm, symbol Isolator:LTV-356T
- R1, R16, R2: value 10k -> 910; footprint Resistor_SMD:R_0603_1608Metric -> Resistor_SMD:R_0805_2012Metric
- R3: footprint Resistor_SMD:R_0603_1608Metric -> Resistor_SMD:R_0805_2012Metric
Connections:
- net +3V3: no longer R1.1, R16.1, R2.1, R3.1
- net +5V: now also R3.1, R18.1, R21.1, R24.1, R27.1, R30.1, R33.1
- net GND: now also J1.2 (Pin_2), U1.3, U2.3, U4.3, U5.3, U6.3, U7.3, U8.3
- net IN1: now also U3.36 (GPIO22), R33.2, U8.4; no longer R16.2, U3.37 (GPIO23)
- net IN2: now also U3.37 (GPIO23), U1.4; no longer U3.36 (GPIO22)
- net IN3: now also U3.9 (DAC_1/ADC2_CH8/GPIO25), R18.2, U2.4; no longer R2.2, U3.28 (GPIO17)
- net IN4: now also U3.10 (DAC_2/ADC2_CH9/GPIO26), R21.2, U4.4; no longer R1.2, U3.27 (GPIO16)
- net IN5: now reaches U3.11 (ADC2_CH7/GPIO27)
- net IN5: now also R24.2, U5.4
- new net: R25.2, R26.1
- new net: R1.1, R2.2
- new net: R1.2, U1.1
- new net: R28.2, R29.1
- new net: R20.2, U4.1
- new net: R32.2, U8.1
- new net: R22.2, R23.1
- new net: R23.2, U5.1
- new net: R29.2, U7.1
- new net: R26.2, U6.1
- new net: R16.2, R17.1
- new net: R17.2, U2.1
- new net: R31.2, R32.1
- new net: R19.2, R20.1
- new net GND1: J1.1 (Pin_1), J7.1 (Pin_1), U1.2, U2.2, U4.2, U5.2, U6.2, U7.2, U8.2
- new net IN6: R27.2, U3.27 (GPIO16), U6.4
- new net IN7: R30.2, U3.28 (GPIO17), U7.4
- new net IN_T_1: J7.8 (Pin_8), R31.1
- new net IN_T_2: J7.7 (Pin_7), R2.1
- new net IN_T_3: J7.6 (Pin_6), R16.1
- new net IN_T_4: J7.5 (Pin_5), R19.1
- new net IN_T_5: J7.4 (Pin_4), R22.1
- new net IN_T_6: J7.3 (Pin_3), R25.1
- new net IN_T_7: J7.2 (Pin_2), R28.1
Other:
- moved on the sheet: J6

Commit message: Update Schematic
Parts:
- added C1: 1uF, Capacitor_SMD:C_0603_1608Metric, symbol Device:C
- added C2: 10nF, Capacitor_SMD:C_0603_1608Metric, symbol Device:C
- added D15, D16, D17, D18, D19: LED, LED_SMD:LED_0603_1608Metric, symbol Device:LED
- added J10: CT_CLAMP_K2, Connector_PinHeader_2.54mm:PinHeader_1x02_P2.54mm_Vertical, symbol Connector:Conn_01x02_Pin
- added J11: CT_CLAMP_K3, Connector_PinHeader_2.54mm:PinHeader_1x02_P2.54mm_Vertical, symbol Connector:Conn_01x02_Pin
- added J12: CT_CLAMP_K4, Connector_PinHeader_2.54mm:PinHeader_1x02_P2.54mm_Vertical, symbol Connector:Conn_01x02_Pin
- added J13: CT_CLAMP_K5, Connector_PinHeader_2.54mm:PinHeader_1x02_P2.54mm_Vertical, symbol Connector:Conn_01x02_Pin
- added J9: Lamp_AC, TerminalBlock:TerminalBlock_MaiXu_MX126-5.0-02P_1x02_P5.00mm, symbol Connector:Screw_Terminal_01x02
- added Q6: BT136-600, Package_TO_SOT_THT:TO-220-3_Vertical, symbol Triac_Thyristor:BT136-600
- added Q7: MMBT2222A, Package_TO_SOT_SMD:SOT-23, symbol Transistor_BJT:MMBT2222A
- added R34, R35: 10k, Resistor_SMD:R_0603_1608Metric, symbol Device:R
- added R36, R37, R38, R39: 33, Resistor_SMD:R_0603_1608Metric, symbol Device:R
- added R40: 1K, Resistor_SMD:R_0603_1608Metric, symbol Device:R
- added R41: 330, Resistor_SMD:R_0603_1608Metric, symbol Device:R
- added R42: 220, Resistor_SMD:R_0603_1608Metric, symbol Device:R
- added R43: 100, Resistor_SMD:R_0805_2012Metric, symbol Device:R
- added R44, R45, R46, R47, R48: 1k, Resistor_SMD:R_0603_1608Metric, symbol Device:R
- added U10, U12: 74LVC2G08, Package_TO_SOT_SMD:SOT-23-8, symbol 74xGxx:74LVC2G08
- added U11, U9: 74LVC2G04, Package_TO_SOT_SMD:SOT-23-6, symbol 74xGxx:74LVC2G04
- added U20: MOC3041M, Package_DIP:DIP-6_W7.62mm, symbol Relay_SolidState:MOC3041M
- U3: footprint PCM_Espressif:ESP32-DevKitC -> GateLinkMaster_Local:ESP32-DevKitC-Local
Connections:
- net +3V3: now also R34.1, U10.8 (VCC), U11.5 (VCC), U12.8 (VCC), U9.5 (VCC)
- net +5V: now also R41.1
- net GND: now also C1.2, D15.1 (K), D16.1 (K), D17.1 (K), D18.1 (K), D19.1 (K), Q7.2 (E), R35.2, U10.4 (GND), U11.2 (GND), U12.4 (GND), U9.2 (GND)
- net SIG1: now also U10.1, U9.3; no longer R7.1
- net SIG2: now also U10.5, U9.1; no longer R4.1
- net SIG3: now also U11.3, U12.1; no longer R10.1
- net SIG4: now also U11.1, U12.5; no longer R13.1
- net at J2.2 (Pin_2), K2.1: now also J3.2 (Pin_2), J3.3 (Pin_3), K3.1, K3.4
- net LAMP_BLINK: now reaches U3.12 (MTMS/GPIO14/ADC2_CH6)
- net LAMP_BLINK: now also R40.1, R48.1
- net I_K2_SENSE: now reaches U3.5 (VDET_1/GPIO34/ADC1_CH6)
- net I_K2_SENSE: now also J10.1 (Pin_1), R36.1
- net I_K3_SENSE: now reaches U3.6 (VDET_2/GPIO35/ADC1_CH7)
- net I_K3_SENSE: now also J11.1 (Pin_1), R37.1
- net I_K4_SENSE: now reaches U3.7 (32K_XP/GPIO32/ADC1_CH4)
- net I_K4_SENSE: now also J12.1 (Pin_1), R38.1
- net I_K5_SENSE: now reaches U3.8 (32K_XN/GPIO33/ADC1_CH5)
- net I_K5_SENSE: now also J13.1 (Pin_1), R39.1
- new net: Q7.3 (C), R41.2, U20.1, U20.2
- new net: C2.2, J9.2 (Pin_2), Q6.1 (A1), Q6.3 (G), R42.2, U20.4
- new net: R42.1, U20.6
- new net: D19.2 (A), R48.2
- new net: J9.1 (Pin_1), Q6.2 (A2), R43.1
- new net: C2.1, R43.2
- new net: D17.2 (A), R46.2
- new net: D16.2 (A), R45.2
- new net: Q7.1 (B), R40.2
- new net: D15.2 (A), R44.2
- new net: D18.2 (A), R47.2
- new net ADC_BIAS: C1.1, J10.2 (Pin_2), J11.2 (Pin_2), J12.2 (Pin_2), J13.2 (Pin_2), R34.2, R35.1, R36.2, R37.2, R38.2, R39.2
- new net NOT_SIG1: U10.6, U9.4
- new net NOT_SIG2: U10.2, U9.6
- new net NOT_SIG3: U11.4, U12.6
- new net NOT_SIG4: U11.6, U12.2
- new net SIG1_EN: R44.1, R7.1, U10.7
- new net SIG2_EN: R4.1, R45.1, U10.3
- new net SIG3_EN: R10.1, R46.1, U12.7
- new net SIG4_EN: R13.1, R47.1, U12.3
Other:
- added sheet ESP32_MasterBoard (ESP32_MasterBoard.kicad_sch)
- note added: "U3 = 2x19 socket (DevKitC pinout), NOT a soldered chip.\nAny pin-compatible ESP32 board plugs in here -\nsee the Master/Test-Board sheet for the board we actually populate it with."
